File: pcbdemo1/pcbdemo1.kicad_pcb (KiCad board)
At the start: 2 copper layers, 80 x 51 mm, 88 parts, among them J1 motor, J2 power12V, J3 USB_C_Receptacle_USB2.0, J4 Micro_SD_Card, J5 speedA, J6 speedB, J7 ADC, Q1 BC846, Q2 BC846, Q3 NPN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

Commit message: updata PCB Signed-off-by: fong <wuwenfengmi@outlook.com>
Parts:
- removed D2: 1N4148W, Diode_SMD:D_SOD-123
- added U9: LM1117MP-5.0, Package_TO_SOT_SMD:SOT-223-3_TabPin2, F.Cu at (123.8, 72.8)
- Q6: value NPN -> PNP
- Q7: value PNP -> NPN
- R13, R14, R15, R16, R17, R18, R19, R20, R21, R22, R23, R24, R25, R26, R27, R28, R29, R30, R31, R32, R33, R34: footprint Resistor_SMD:R_0201_0603Metric -> Resistor_SMD:R_0603_1608Metric
- U2, U3, U4: footprint Package_SO:SOP-8_5.28x5.23mm_P1.27mm -> Package_SO:SOP-8_3.76x4.96mm_P1.27mm
- moved U5 12.5 mm to (114.3, 72.7)
- moved R19 5.60 mm to (77.8, 54.4), turned to 90 degrees
- moved R16 5.53 mm to (77.8, 65.0), turned to 90 degrees
- moved R21 5.50 mm to (77.7, 61.8), turned to 90 degrees
- moved Q6 4.81 mm to (74.6, 61.8)
- moved R20 4.80 mm to (77.1, 50.7), turned to 90 degrees
- moved R22 3.92 mm to (76.2, 57.9), turned to 90 degrees
- moved R15 3.81 mm to (76.1, 69.2), turned to 90 degrees
- moved R32 3.75 mm to (78.6, 67.7)
- moved R29 3.63 mm to (79.7, 54.4), turned to 90 degrees
- moved TP2 3.01 mm to (70.4, 49.9)
- moved Q7 2.50 mm to (74.8, 65.4)
- moved Q5 2.33 mm to (72.9, 69.3)
- moved R31 2.32 mm to (79.5, 65.0), turned to -90 degrees
- moved R26 2.20 mm to (77.8, 76.4)
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Connections:
- C1 pad 1: +12V -> /USB_VDD
- Q3 pad 1: Net-(Q3-C) -> Net-(Q3-B)
- Q3 pad 2: Net-(Q3-B) -> GND
- Q3 pad 3: GND -> Net-(Q3-C)
- Q4 pad 1: Net-(Q4-C) -> Net-(Q4-B)
- Q4 pad 2: Net-(Q4-B) -> +12V
- Q4 pad 3: +12V -> Net-(Q4-C)
- Q5 pad 1: Net-(Q5-C) -> Net-(Q5-B)
- Q5 pad 2: Net-(Q5-B) -> +12V
- Q5 pad 3: +12V -> Net-(Q5-C)
- Q6 pad 1: Net-(Q6-C) -> Net-(Q6-B)
- Q6 pad 2: Net-(Q6-B) -> +12V
- Q6 pad 3: GND -> Net-(Q6-C)
- Q7 pad 1: Net-(Q7-C) -> Net-(Q7-B)
- Q7 pad 2: Net-(Q7-B) -> GND
- Q7 pad 3: +12V -> Net-(Q7-C)
- Q8 pad 1: Net-(Q8-C) -> Net-(Q8-B)
- Q8 pad 2: Net-(Q8-B) -> GND
- Q8 pad 3: GND -> Net-(Q8-C)
- R16 pad 1: Net-(Q6-B) -> Net-(Q7-B)
- R18 pad 2: Net-(Q6-C) -> Net-(Q7-C)
- R21 pad 1: Net-(Q7-B) -> Net-(Q6-B)
- R23 pad 2: Net-(Q7-C) -> Net-(Q6-C)
- R30 pad 2: Net-(Q7-B) -> Net-(Q6-B)
- R31 pad 2: Net-(Q6-B) -> Net-(Q7-B)
- TP4 pad 1: Net-(Q6-C) -> Net-(Q7-C)
- TP5 pad 1: Net-(Q7-C) -> Net-(Q6-C)
- U3 pad 4: Net-(Q6-C) -> Net-(Q7-C)
- U4 pad 2: Net-(Q7-C) -> Net-(Q6-C)
- U5 pad 3: +12V -> /USB_VDD
Routing:
- net /USB_VDD: track 19.0 -> 71.3 mm
- net +12V: track 176.7 -> 142.7 mm
- net Net-(Q3-B): track 12.7 -> 5.76 mm
- net Net-(Q4-B): track 10.6 -> 3.70 mm
- net VCC: track 237.0 -> 243.8 mm
- net Net-(Q5-B): track 11.3 -> 5.17 mm
- net /EN_C: track 34.9 -> 39.5 mm
- net Net-(Q6-C): track 13.5 -> 9.06 mm
- net GND: track 531.4 -> 527.3 mm, vias 4 -> 5
- net Net-(Q6-B): track 8.44 -> 4.50 mm
- net Net-(Q8-B): track 7.75 -> 3.83 mm
- net Net-(Q7-B): track 7.04 -> 3.78 mm
- net Net-(Q8-C): track 11.2 -> 8.37 mm
- net Net-(Q4-C): track 10.1 -> 7.28 mm
- net Net-(U7-IO32): track 2.72 -> 5.20 mm
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Other:
- board text added: "Motor Controller V0.99 Designed by kevin 2023-05-20 https://lmve.net https://wnfed.com"
- board text removed: "Motor Controller Designed by kevin 2023-05-07 https://lmve.net Blog: https://wnfed.com"
