File: pcbdemo1/pcbdemo1.kicad_sch (KiCad schematic)
At the start: 88 parts, among them J1 motor, J2 power12V, J3 USB_C_Receptacle_USB2.0, J4 Micro_SD_Card, J5 speedA, J6 speedB, J7 ADC, Q1 BC846, Q2 BC846, Q3 NPN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

Commit message: updata PCB Signed-off-by: fong <wuwenfengmi@outlook.com>
Parts:
- removed D2: 1N4148W, Diode_SMD:D_SOD-123, symbol Diode:1N4148W
- removed Q6: NPN, Package_TO_SOT_SMD:SOT-23-3, symbol Simulation_SPICE:NPN
- removed Q7: PNP, Package_TO_SOT_SMD:SOT-23-3, symbol Simulation_SPICE:PNP
- added Q6: PNP, Package_TO_SOT_SMD:SOT-23-3, symbol Simulation_SPICE:PNP
- added Q7: NPN, Package_TO_SOT_SMD:SOT-23-3, symbol Simulation_SPICE:NPN
- added U9: LM1117MP-5.0, Package_TO_SOT_SMD:SOT-223-3_TabPin2, symbol Regulator_Linear:LM1117MP-5.0
- R13, R14, R15, R16, R17, R18, R19, R20, R21, R22, R23, R24, R25, R26, R27, R28, R29, R30, R31, R32, R33, R34: footprint Resistor_SMD:R_0201_0603Metric -> Resistor_SMD:R_0603_1608Metric
- U2, U3, U4: footprint Package_SO:SOP-8_5.28x5.23mm_P1.27mm -> Package_SO:SOP-8_3.76x4.96mm_P1.27mm
Connections:
- net +12V: now also Q4.2 (E), Q5.2 (E), Q6.2 (E), U9.3 (VI); no longer C1.1, Q4.3 (E), Q5.3 (E), U5.3 (VI)
- net GND: now also Q3.2 (E), Q8.2 (E), Q7.2 (E), U9.1 (GND); no longer Q3.3 (E), Q8.3 (E)
- net USB_VDD: now also C1.1, U5.3 (VI), U9.2 (VO)
- net at R17.2, TP3.1, U3.2 (g1): now also Q5.3 (C); no longer Q5.1 (C)
- net at R15.1, R32.2: now also Q5.1 (B); no longer Q5.2 (B)
- net at R18.2, TP4.1, U3.4 (g2): now also Q7.3 (C)
- net at R24.2, TP6.1, U4.4 (g2): now also Q8.3 (C); no longer Q8.1 (C)
- net at R22.1, R34.2: now also Q8.1 (B); no longer Q8.2 (B)
- net at R16.1, R31.2: now also Q7.1 (B)
- net at R13.2, TP1.1, U2.2 (g1): now also Q4.3 (C); no longer Q4.1 (C)
- net at R19.1, R33.2: now also Q4.1 (B); no longer Q4.2 (B)
- net at R21.1, R30.2: now also Q6.1 (B)
- net at R23.2, TP5.1, U4.2 (g1): now also Q6.3 (C)
- net at R14.2, TP2.1, U2.4 (g2): now also Q3.3 (C); no longer Q3.1 (C)
- net at R20.1, R29.2: now also Q3.1 (B); no longer Q3.2 (B)
Other:
- moved on the sheet: C1, J2
